File: casino-chip.kicad_pcb (KiCad board)
At the start: 2 copper layers, 0 parts

Commit message: finished generic chip design (no decorations)
Routing:
- net (no net): vias 0 -> 1
Other:
- board outline added: 43 x 43 mm
